File: pcb_layout/_autosave-thesis_custom_arduino_board.kicad_pcb (KiCad board)
At the start: 2 copper layers, 84.2 x 86.4 mm, 40 parts, among them J1 POWER, J10 RPI VIN, J11 LN DETECT, J12 RELAY VIN, J13 6-CHANNEL RELAY, J2 USB to TTL, J3 ICSP, J4 VSupply, J5 Physical Buttons, J6 VSupply, J7 Light Sensor, J8 J8, J9 RPi Connector, M1 TXB0104, M2 TB6612FNG, M3 GY-906-BCC, M4 JSN-SR04T, SW1 Reset SW, U1 ATmega328P-P, U2 LM7805, U3 LM317, Y1 16MHz

Commit message: PCB layout: Revision 3.0
Parts:
- added J14: DSI VIN, Connector_JST:JST_XH_B2B-XH-A_1x02_P2.50mm_Vertical, F.Cu at (178.6, 135.9)
- J8: value J8 -> I2C Device
- moved J5 6.30 mm to (175.8, 143.6), turned to 0 degrees
- moved MTR1 2.84 mm to (178.6, 127.8), turned to 0 degrees
- renumbered MTR to MTR1
Connections:
- U1 pad 14: /D8 -> unconnected-(U1-PB0-Pad14)
- U1 pad 24: /A1 -> unconnected-(U1-PC1-Pad24)
- U1 pad 25: /A2 -> unconnected-(U1-PC2-Pad25)
- U1 pad 26: /A3 -> unconnected-(U1-PC3-Pad26)
Routing:
- net VDC: track 24.2 -> 82.2 mm
- net /mtr_l1: track 22.6 -> 19.8 mm
- net /BTN2: track 43.5 -> 41.3 mm
- net /mtr_l2: track 22.6 -> 24.0 mm
- net VCC: track 257.1 -> 256.2 mm
- net /BTN1: track 14.7 -> 14.0 mm
